File: hardware/usb.kicad_sch (KiCad schematic)
At the start: 5 parts

Commit message: Audio circuit layout
Parts:
- removed C25: 100n, Capacitor_SMD:C_0402_1005Metric, symbol Device:C
- removed D9: USBLC6-2SC6, _lib:SOT-23-6_L2.9-W1.6-P0.95-LS2.8-BL, symbol _lib:USBLC6-2SC6
- removed R19, R20: 5.1k, Resistor_SMD:R_0402_1005Metric, symbol Device:R
- removed USB1: TYPE-C 16PIN 2MD(073), _lib:USB-C-SMD_TYPE-C-16PIN, symbol _lib:USB-C-SMD_TYPE-C-16PIN
Connections:
- no-connect marks 2 -> 0
