File: hardware/squishbox_zero.kicad_pcb (KiCad board)
At the start: 4 copper layers, 21 parts, among them J1 PPS_UFL, J2 PPS_SMA, J3 LED, J4 UART_HDR, U1 XC6206P332MR-G

Commit message: Rough form factor in place
Parts:
- removed J2: PPS_SMA, Connector_Coaxial:SMA_Samtec_SMA-J-P-H-ST-EM1_EdgeMount
- added A1: Raspberry Pi Zero, _lib:Raspberry_Pi_Zero, B.Cu at (117.6, 85.2)
- added J5: USB_A, _lib:USB-A-SMD_USB-M-21, B.Cu at (123.5, 100.0)
- added U2: PCM5102A, Package_SO:TSSOP-20_4.4x6.5mm_P0.65mm, B.Cu at (159.4, 97.8)
- J1: value PPS_UFL -> AudioJack4_SwitchTR1; footprint _lib:IPEX-SMD_HC-RF-IPEX0303-01 -> _lib:AUDIO-SMD_PJ-342; moved to B.Cu
- USB1: moved to B.Cu
- moved C25 90.1 mm to (205.1, 100.4)
- moved D9 90.1 mm to (198.7, 101.6)
- moved R19 90.1 mm to (202.2, 100.4)
- moved R20 90.1 mm to (202.2, 102.4)
- moved C1 76.6 mm to (107.4, 164.5)
- moved D2 76.6 mm to (107.2, 152.8)
- moved TP1 76.6 mm to (107.2, 167.6)
- moved C2 76.6 mm to (106.8, 170.3)
- moved C3 76.6 mm to (106.8, 172.3)
- moved D1 76.6 mm to (107.2, 149.8)
- moved D3 76.6 mm to (107.2, 155.7)
- moved D4 76.6 mm to (102.2, 154.7)
- moved H1 76.6 mm to (101.4, 161.4)
- moved H2 76.6 mm to (101.4, 169.3)
- moved J3 76.6 mm to (107.5, 159.1)
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Other:
- board outline added: 65 x 30 mm
- copper layers 4 -> 2

Commit message: Audio circuit layout
Parts:
- removed C25: 100n, Capacitor_SMD:C_0402_1005Metric
- removed D2: BAT60JFILM, Diode_SMD:D_SOD-323
- removed H1, H2: MountingHole_Pad, MountingHole:MountingHole_3.2mm_M3_Pad
- removed J4: UART_HDR, Connector_PinHeader_2.54mm:PinHeader_1x04_P2.54mm_Horizontal
- removed JP1: PWR_SELECT, Jumper:SolderJumper-3_P1.3mm_Open_RoundedPad1.0x1.5mm_NumberLabels
- removed TP1: 5V_EXT, TestPoint:TestPoint_Pad_D1.5mm
- added C10: 2.2n, Capacitor_SMD:C_0402_1005Metric, F.Cu at (132.1, 164.5)
- added C11: 10u, Capacitor_SMD:C_0603_1608Metric, F.Cu at (135.6, 170.4)
- added C12: 100n, Capacitor_SMD:C_0402_1005Metric, F.Cu at (132.1, 166.5)
- added C26: 100n, Capacitor_SMD:C_0402_1005Metric, F.Cu at (132.1, 168.5)
- added C4: 100n, Capacitor_SMD:C_0402_1005Metric, F.Cu at (122.8, 142.3)
- added C5: 2.2u, Capacitor_SMD:C_0402_1005Metric, F.Cu at (122.8, 144.2)
- added C6: 2.2u, Capacitor_SMD:C_0402_1005Metric, F.Cu at (132.1, 158.6)
- added C7: 2.2n, Capacitor_SMD:C_0402_1005Metric, F.Cu at (132.1, 160.6)
- added C8: 10u, Capacitor_SMD:C_0603_1608Metric, F.Cu at (135.6, 167.9)
- added C9: 100n, Capacitor_SMD:C_0402_1005Metric, F.Cu at (132.1, 162.6)
- added R21: 470, Resistor_SMD:R_0402_1005Metric, F.Cu at (129.2, 162.6)
- added R22: 470, Resistor_SMD:R_0402_1005Metric, F.Cu at (129.2, 164.6)
- added R23: 22, Resistor_SMD:R_0402_1005Metric, F.Cu at (129.2, 166.6)
- added R24: 22, Resistor_SMD:R_0402_1005Metric, F.Cu at (129.2, 168.6)
- added R25: 22, Resistor_SMD:R_0402_1005Metric, F.Cu at (129.2, 170.6)
- J1: value AudioJack4_SwitchTR1 -> LINE OUT
- J5: value USB_A -> USB_HOST
- U1: moved to B.Cu
- moved U1 96.0 mm to (159.5, 103.5), turned to 180 degrees
- moved R20 93.4 mm to (129.2, 160.6)
- moved R19 93.4 mm to (129.2, 158.6)
- moved D9 89.2 mm to (140.1, 168.8)
- moved USB1 0.53 mm to (177.9, 103.5)
Connections:
- net /USB/USB_CC1 renamed /USB_CC1
- net /USB/USB_CC2 renamed /USB_CC2
- A1 pad 1: unconnected-(A1-+3V3-Pad1) -> +3V3D
- A1 pad PP1: unconnected-(A1-+5V_USB-PadPP1) -> /V_USB_HOST
- A1 pad PP22: unconnected-(A1-USB_D+-PadPP22) -> /USB_D_HOST_P
- A1 pad PP23: unconnected-(A1-USB_D--PadPP23) -> /USB_D_HOST_N
- A1 pad PP6: unconnected-(A1-GND-PadPP6) -> GND
- C1 pad 1: +5V -> +3V3A
- C3 pad 1: +3V3 -> unconnected-(C3-Pad1)
- C3 pad 2: GND -> unconnected-(C3-Pad2)
- D1 pad 1: +5V -> +5V_USB
- D1 pad 2: unconnected-(D1-A-Pad2) -> Net-(D1-A)
- D3 pad 2: +3V3 -> +3V3A
- D9 pad 1: /USB/USB_D_CONN_N -> /USB_D_HOST_P
- D9 pad 3: /USB/USB_D_CONN_P -> /USB_D_HOST_N
- D9 pad 4: /USB/USB_D_P -> /USB_D_N
- D9 pad 5: +5V_USB -> unconnected-(D9-VBUS-Pad5)
- D9 pad 6: /USB/USB_D_N -> /USB_D_P
- J1 pad R1: unconnected-(J1-PadR1) -> Net-(C7-Pad1)
- J1 pad S: unconnected-(J1-PadS) -> GND
- J1 pad T: unconnected-(J1-PadT) -> Net-(C10-Pad1)
- J5 pad 1: unconnected-(J5-VBUS-Pad1) -> /V_USB_HOST
- J5 pad 2: unconnected-(J5-D--Pad2) -> /USB_D_N
- J5 pad 3: unconnected-(J5-D+-Pad3) -> /USB_D_P
- J5 pad 4: unconnected-(J5-GND-Pad4) -> GND
- J5 pad 5: unconnected-(J5-Shield-Pad5) -> GND
- U1 pad 2: +3V3 -> +3V3A
- U2 pad 1: unconnected-(U2-CPVDD-Pad1) -> +3V3A
- U2 pad 10: unconnected-(U2-DEMP-Pad10) -> GND
- U2 pad 11: unconnected-(U2-FLT-Pad11) -> +3V3D
- U2 pad 12: unconnected-(U2-SCK-Pad12) -> GND
- U2 pad 13: unconnected-(U2-BCK-Pad13) -> /I2S_CLK
- U2 pad 14: unconnected-(U2-DIN-Pad14) -> /I2S_DATA
- U2 pad 15: unconnected-(U2-LRCK-Pad15) -> /I2S_WS
- U2 pad 16: unconnected-(U2-FMT-Pad16) -> GND
- U2 pad 17: unconnected-(U2-XSMT-Pad17) -> +3V3D
- U2 pad 18: unconnected-(U2-LDOO-Pad18) -> Net-(U2-LDOO)
- U2 pad 19: unconnected-(U2-DGND-Pad19) -> GND
- U2 pad 2: unconnected-(U2-CAPP-Pad2) -> Net-(U2-CAPP)
- U2 pad 20: unconnected-(U2-DVDD-Pad20) -> +3V3D
- U2 pad 3: unconnected-(U2-CPGND-Pad3) -> GND
- U2 pad 4: unconnected-(U2-CAPM-Pad4) -> Net-(U2-CAPM)
- U2 pad 5: unconnected-(U2-VNEG-Pad5) -> Net-(U2-VNEG)
- U2 pad 6: unconnected-(U2-OUTL-Pad6) -> Net-(U2-OUTL)
- U2 pad 7: unconnected-(U2-OUTR-Pad7) -> Net-(U2-OUTR)
- U2 pad 8: unconnected-(U2-AVDD-Pad8) -> +3V3A
- U2 pad 9: unconnected-(U2-AGND-Pad9) -> GND
- USB1 pad 11: +5V_USB -> Net-(D1-A)
- USB1 pad 2: +5V_USB -> Net-(D1-A)
- USB1 pad 5: /USB/USB_D_CONN_N -> unconnected-(USB1-DN2-Pad5)
- USB1 pad 6: /USB/USB_D_CONN_P -> unconnected-(USB1-DP1-Pad6)
- USB1 pad 7: /USB/USB_D_CONN_N -> unconnected-(USB1-DN1-Pad7)
- USB1 pad 8: /USB/USB_D_CONN_P -> unconnected-(USB1-DP2-Pad8)

Commit message: LCD + Finalised Schematic
Parts:
- removed the C3 at (106.8, 172.3)
- removed D3: BAT60JFILM, Diode_SMD:D_SOD-323
- removed D4: WS2812B-2020, LED_SMD:LED_WS2812B-2020_PLCC4_2.0x2.0mm
- removed J3: LED, Connector_PinHeader_1.27mm:PinHeader_1x03_P1.27mm_Vertical
- added FB1: GZ1608D601TF, Resistor_SMD:R_0603_1608Metric, B.Cu at (130.8, 96.5)
- added JP1: SLOW_FILT, Jumper:SolderJumper-2_P1.3mm_Open_RoundedPad1.0x1.5mm, B.Cu at (146.2, 104.5)
- added R6: 10k, Resistor_SMD:R_0402_1005Metric, B.Cu at (144.2, 102.0)
- added U1: ~, _lib:SSD1306-0.91-OLED-4pin-128x32, B.Cu at (130.5, 106.0)
- C1: renamed from C2; moved to B.Cu
- C10: renamed from C9; moved to B.Cu
- C11: renamed from C7; moved to B.Cu
- C12: renamed from C10; moved to B.Cu
- C2: renamed from C26; moved to B.Cu
- C3: renamed from C1; moved to B.Cu
- C4, D1: moved to B.Cu
- C5: renamed from C6; moved to B.Cu
- C6: renamed from C11; moved to B.Cu
- C7: renamed from C12; moved to B.Cu
- C8: renamed from C5; moved to B.Cu
- C9: renamed from C8; moved to B.Cu
- D2: renamed from D9; moved to B.Cu
- R1: renamed from R25; moved to B.Cu
- R2: renamed from R19; moved to B.Cu
- R3: renamed from R20; moved to B.Cu
- R4: renamed from R24; moved to B.Cu
- R5: renamed from R23; moved to B.Cu
- R7: renamed from R21; moved to B.Cu
- R8: renamed from R22; moved to B.Cu
- moved C1 84.1 mm to (159.8, 105.0), turned to 180 degrees
- moved C12 81.9 mm to (167.2, 90.5), turned to 90 degrees
- moved R8 81.3 mm to (165.8, 92.0)
- moved R7 80.4 mm to (165.8, 91.0)
- moved C3 79.1 mm to (156.8, 102.8), turned to -90 degrees
- moved D1 78.8 mm to (173.0, 106.5)
- moved C11 76.6 mm to (167.3, 92.5), turned to -90 degrees
- moved C6 76.1 mm to (144.0, 94.8), turned to 180 degrees
- moved R3 73.1 mm to (173.5, 102.5), turned to 180 degrees
- moved C7 71.5 mm to (144.2, 96.0), turned to 180 degrees
- moved C2 70.8 mm to (131.1, 97.7), turned to 180 degrees
- moved C9 70.1 mm to (143.8, 98.2), turned to 180 degrees
- moved R2 69.5 mm to (173.5, 105.0), turned to 180 degrees
- moved D2 69.5 mm to (131.2, 100.0), turned to 90 degrees
- moved R4 67.1 mm to (159.0, 108.5), turned to 180 degrees
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- renumbered J5 to J1, J1 to J2, U1 to U2, U2 to U3
Connections:
- net Net-(C10-Pad1) renamed /DAC_OUTL_FILT
- net Net-(C7-Pad1) renamed /DAC_OUTR_FILT
- net Net-(D1-A) renamed /USB_VBUS
- net Net-(U2-CAPM) renamed /DAC_CAPM
- net Net-(U2-CAPP) renamed /DAC_CAPP
- net Net-(U2-LDOO) renamed /DAC_LDO
- net Net-(U2-OUTL) renamed /DAC_OUTL
- net Net-(U2-OUTR) renamed /DAC_OUTR
- net Net-(U2-VNEG) renamed /DAC_VNEG
- A1 pad 12: unconnected-(A1-GP18-Pad12) -> /I2S_CLK_SOC
- A1 pad 14: unconnected-(A1-GND-Pad14) -> GND
- A1 pad 17: unconnected-(A1-+3V3-Pad17) -> +3V3D
- A1 pad 2: unconnected-(A1-+5V-Pad2) -> +5V
- A1 pad 20: unconnected-(A1-GND-Pad20) -> GND
- A1 pad 25: unconnected-(A1-GND-Pad25) -> GND
- A1 pad 3: unconnected-(A1-GP2/SDA-Pad3) -> /OLED_SDA
- A1 pad 30: unconnected-(A1-GND-Pad30) -> GND
- A1 pad 34: unconnected-(A1-GND-Pad34) -> GND
- A1 pad 35: unconnected-(A1-GP19-Pad35) -> /I2S_WS_SOC
- A1 pad 39: unconnected-(A1-GND-Pad39) -> GND
- A1 pad 4: unconnected-(A1-+5V-Pad4) -> +5V
- A1 pad 40: unconnected-(A1-GP21-Pad40) -> /I2S_DATA_SOC
- A1 pad 5: unconnected-(A1-GP3/SCL-Pad5) -> /OLED_SCL
- A1 pad 6: unconnected-(A1-GND-Pad6) -> GND
- A1 pad 9: unconnected-(A1-GND-Pad9) -> GND
- C2 pad 1: unconnected-(C26-Pad1) -> /V_USB_HOST
- D1 pad 1: +5V_USB -> +5V
- D2 pad 1: /USB_D_HOST_P -> /USB_D_P
- D2 pad 3: /USB_D_HOST_N -> /USB_D_N
- D2 pad 4: /USB_D_N -> /USB_D_HOST_N
- D2 pad 5: unconnected-(D9-VBUS-Pad5) -> /V_USB_HOST
- D2 pad 6: /USB_D_P -> /USB_D_HOST_P
- J1 pad 1: /V_USB_HOST -> /V_USB_HOST_FB
- R1 pad 1: unconnected-(R25-Pad1) -> /I2S_WS
- R1 pad 2: unconnected-(R25-Pad2) -> /I2S_WS_SOC
- R4 pad 1: unconnected-(R24-Pad1) -> /I2S_CLK_SOC
- R4 pad 2: unconnected-(R24-Pad2) -> /I2S_CLK
- R5 pad 1: unconnected-(R23-Pad1) -> /I2S_DATA_SOC
- R5 pad 2: unconnected-(R23-Pad2) -> /I2S_DATA
- U3 pad 11: +3V3D -> /DAC_FLT
Routing:
- net /I2S_WS: track 0.00 -> 18.2 mm
- net /OLED_SDA: track 0.00 -> 16.2 mm
- net /V_USB_HOST: track 0.00 -> 14.9 mm
- net /OLED_SCL: track 0.00 -> 12.6 mm
- net /I2S_DATA_SOC: track 0.00 -> 8.60 mm
- net /I2S_CLK_SOC: track 0.00 -> 5.62 mm
- net +3V3D: track 0.00 -> 4.84 mm
- net /USB_D_P: track 0.00 -> 2.80 mm
- net /USB_D_N: track 0.00 -> 2.76 mm
- net /V_USB_HOST_FB: track 0.00 -> 2.69 mm
- net +5V: track 0.00 -> 2.54 mm
- net /I2S_WS_SOC: track 0.00 -> 1.96 mm
- net /USB_CC2: track 0.00 -> 1.63 mm
- net /USB_CC1: track 0.00 -> 1.63 mm

Commit message: Routed
Parts:
- added G***: LOGO, _lib:BOJIT_LOGO, B.Cu at (153.2, 88.8)
- added kibuzzard-68B38B7F: G***, kibuzzard-68B38B7F, B.Cu at (143.2, 104.2)
- moved R5 4.58 mm to (132.3, 108.0), turned to 90 degrees
- moved R6 4.13 mm to (148.1, 103.5), turned to -90 degrees
- moved R4 1.80 mm to (157.5, 107.5)
- moved R2 1.00 mm to (173.5, 104.0)
- moved R1 0.71 mm to (131.0, 108.0), turned to -90 degrees
- moved D1 0.50 mm to (173.5, 106.5), turned to 90 degrees
- moved USB1 0.50 mm to (177.9, 103.0)
- moved C5 0.35 mm to (154.5, 98.5)
- moved C8 0.35 mm to (154.0, 97.0)
- moved JP1 0.25 mm to (146.2, 104.2)
- moved C6 0.12 mm to (143.9, 94.7)
- moved C9 0.10 mm to (143.8, 98.3)
Connections:
- A1 pad 1: +3V3D -> unconnected-(A1-+3V3-Pad1)
Routing:
- net GND: track 0.00 -> 54.2 mm, vias 0 -> 76
- net +5V: track 2.54 -> 33.8 mm, vias 0 -> 1
- net /I2S_CLK: track 0.00 -> 25.6 mm
- net +3V3D: track 4.84 -> 24.9 mm, vias 0 -> 1
- net /USB_D_HOST_N: track 0.00 -> 19.0 mm
- net /USB_D_HOST_P: track 0.00 -> 18.2 mm, vias 0 -> 1
- net /I2S_DATA: track 0.00 -> 17.7 mm
- net /DAC_OUTL: track 0.00 -> 16.6 mm
- net /DAC_OUTR: track 0.00 -> 16.4 mm
- net +3V3A: track 0.00 -> 15.7 mm
- net /DAC_OUTR_FILT: track 0.00 -> 13.6 mm
- net /USB_VBUS: track 0.00 -> 12.2 mm
- net /DAC_OUTL_FILT: track 0.00 -> 9.42 mm
- net /DAC_FLT: track 0.00 -> 3.75 mm
- net /DAC_LDO: track 0.00 -> 3.15 mm
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- added copper zone on B.Cu, net GND
- added copper zone on F.Cu, net GND

Commit message: First attempt at fab files
Parts:
- C11, C12: footprint Capacitor_SMD:C_0402_1005Metric -> Capacitor_SMD:C_0805_2012Metric
- moved C12 1.77 mm to (168.5, 89.2), turned to 180 degrees
- moved C11 1.26 mm to (168.5, 92.8), turned to 180 degrees
- moved R7 0.50 mm to (165.8, 90.5)
- moved R8 0.50 mm to (165.8, 91.5)
Routing:
- net /DAC_OUTR_FILT: track 13.6 -> 14.9 mm
- net /V_USB_HOST: track 14.9 -> 13.8 mm
- net /DAC_OUTL_FILT: track 9.42 -> 10.3 mm
- net +5V: track 33.8 -> 32.9 mm
- net /I2S_WS: track 19.3 -> 18.8 mm
- net GND: track 54.2 -> 53.7 mm, vias 76 -> 77
