File: hardware/squishbox_zero.kicad_sch (KiCad schematic)
At the start: 16 parts, among them J1 PPS_UFL, J2 PPS_SMA, J3 LED, J4 UART_HDR, U1 XC6206P332MR-G

Commit message: Rough form factor in place
Parts:
- removed J1: PPS_UFL, _lib:IPEX-SMD_HC-RF-IPEX0303-01, symbol _lib:Conn_Coaxial_Small
- removed J2: PPS_SMA, Connector_Coaxial:SMA_Samtec_SMA-J-P-H-ST-EM1_EdgeMount, symbol Connector:Conn_Coaxial
- added A1: Raspberry Pi Zero, _lib:Raspberry_Pi_Zero, symbol _lib:Raspberry_Pi_Zero
- added J1: AudioJack4_SwitchTR1, _lib:AUDIO-SMD_PJ-342, symbol Connector_Audio:AudioJack4_SwitchTR1
- added J5: USB_A, _lib:USB-A-SMD_USB-M-21, symbol Connector:USB_A
- added U2: PCM5102A, Package_SO:TSSOP-20_4.4x6.5mm_P0.65mm, symbol Audio:PCM5102A

Commit message: Audio circuit layout
Parts:
- removed C3: 2.2u, Capacitor_SMD:C_0402_1005Metric, symbol Device:C
- removed D2: BAT60JFILM, Diode_SMD:D_SOD-323, symbol Device:D_Schottky
- removed H1, H2: MountingHole_Pad, MountingHole:MountingHole_3.2mm_M3_Pad, symbol Mechanical:MountingHole_Pad
- removed J3: LED, Connector_PinHeader_1.27mm:PinHeader_1x03_P1.27mm_Vertical, symbol Connector:Conn_01x03_Pin
- removed J4: UART_HDR, Connector_PinHeader_2.54mm:PinHeader_1x04_P2.54mm_Horizontal, symbol Connector:Conn_01x04_Pin
- removed JP1: PWR_SELECT, Jumper:SolderJumper-3_P1.3mm_Open_RoundedPad1.0x1.5mm_NumberLabels, symbol Jumper:SolderJumper_3_Open
- removed TP1: 5V_EXT, TestPoint:TestPoint_Pad_D1.5mm, symbol Connector:TestPoint
- added C10, C7: 2.2n, Capacitor_SMD:C_0402_1005Metric, symbol Device:C
- added C11, C8: 10u, Capacitor_SMD:C_0603_1608Metric, symbol Device:C
- added C12, C26, C4, C9: 100n, Capacitor_SMD:C_0402_1005Metric, symbol Device:C
- added C5, C6: 2.2u, Capacitor_SMD:C_0402_1005Metric, symbol Device:C
- added D9: USBLC6-2SC6, _lib:SOT-23-6_L2.9-W1.6-P0.95-LS2.8-BL, symbol _lib:USBLC6-2SC6
- added R19, R20: 5.1k, Resistor_SMD:R_0402_1005Metric, symbol Device:R
- added R21, R22: 470, Resistor_SMD:R_0402_1005Metric, symbol Device:R
- added R23, R24, R25: 22, Resistor_SMD:R_0402_1005Metric, symbol Device:R
- added USB1: TYPE-C 16PIN 2MD(073), _lib:USB-C-SMD_TYPE-C-16PIN, symbol _lib:USB-C-SMD_TYPE-C-16PIN
- J1: value AudioJack4_SwitchTR1 -> LINE OUT
- J5: value USB_A -> USB_HOST
Connections:
- net +3V3 is gone; now on net +3V3A: D3.2 (A), U1.2 (VO)
- net +5V: no longer C1.1, D1.1 (K)
- net GND: now also A1.PP6 (GND), J1.S, J5.4 (GND), J5.5 (Shield), U2.10 (DEMP), U2.12 (SCK), U2.16 (FMT), U2.19 (DGND), U2.3 (CPGND), U2.9 (AGND), C10.2, C11.2, C12.2, C26.2, C4.2, C6.2, C7.2, C8.2, C9.2, D9.2 (GND), R19.2, R20.2, USB1.1 (GND), USB1.12 (GND), USB1.13 (SHELL)
- net V_USB_HOST: now reaches J5.1 (VBUS)
- net V_USB_HOST: now also A1.PP1 (+5V_USB)
- net USB_D_N: now reaches J5.2 (D-)
- net USB_D_N: now also D9.4 (I/O2)
- net USB_D_P: now reaches J5.3 (D+)
- net USB_D_P: now also D9.6 (I/O1)
- net at D1.2 (A): now also USB1.11 (VBUS), USB1.2 (VBUS)
- net at J1.R1: now also C7.1, R22.2
- net at J1.T: now also C10.1, R21.2
- net +3V3A: now reaches U2.1 (CPVDD)
- net +3V3A: now also C1.1, U2.8 (AVDD), C4.1
- net +3V3D: now reaches U2.11 (FLT)
- net +3V3D: now also A1.1 (+3V3), U2.17 (XSMT), U2.20 (DVDD), C11.1, C12.1
- net I2S_CLK: now reaches U2.13 (BCK)
- net I2S_DATA: now reaches U2.14 (DIN)
- net I2S_WS: now reaches U2.15 (LRCK)
- net at U2.18 (LDOO): now also C8.1, C9.1
- net at U2.2 (CAPP): now also C5.1
- net at U2.4 (CAPM): now also C5.2
- net at U2.5 (VNEG): now also C6.1
- net at U2.6 (OUTL): now also R21.1
- net at U2.7 (OUTR): now also R22.1
- net USB_D_HOST_P: now reaches A1.PP22 (USB_D+)
- net USB_D_HOST_P: now also D9.1 (I/O1)
- net USB_D_HOST_N: now reaches A1.PP23 (USB_D-)
- net USB_D_HOST_N: now also D9.3 (I/O2)
- net LED_STAGE_2: no longer names the net of D4.1 (DOUT)
- new net +5V_USB: D1.1 (K)
- new net USB_CC1: R20.1, USB1.4 (CC1)
- new net USB_CC2: R19.1, USB1.10 (CC2)
- no-connect marks 2 -> 9
Other:
- removed sheet USB
- note added: "COG"
- note added: "Ferrite Bead?"
- note added: "TODO jumper for latency?"
- moved on the sheet: A1, C1, C2, D1, D3, D4, J1, J5, U1, U2

Commit message: LCD + Finalised Schematic
Parts:
- removed D3: BAT60JFILM, Diode_SMD:D_SOD-323, symbol Device:D_Schottky
- removed D4: WS2812B-2020, LED_SMD:LED_WS2812B-2020_PLCC4_2.0x2.0mm, symbol LED:WS2812B-2020
- added FB1: GZ1608D601TF, Resistor_SMD:R_0603_1608Metric, symbol Device:FerriteBead_Small
- added JP1: SLOW_FILT, Jumper:SolderJumper-2_P1.3mm_Open_RoundedPad1.0x1.5mm, symbol Jumper:Jumper_2_Small_Open
- added R6: 10k, Resistor_SMD:R_0402_1005Metric, symbol Device:R
- added U1: ~, _lib:SSD1306-0.91-OLED-4pin-128x32, symbol _lib:OLED_128x32
- renumbered C2 to C1, C9 to C10, C7 to C11, C10 to C12, C26 to C2, C1 to C3, C6 to C5, C11 to C6, C12 to C7, C5 to C8, C8 to C9, D9 to D2, J5 to J1, J1 to J2, R25 to R1, R19 to R2, R20 to R3, R24 to R4, R23 to R5, R21 to R7, R22 to R8, U1 to U2, U2 to U3
Connections:
- net +5V_USB is gone; now on net +5V: D1.1 (K)
- net +3V3D: now also A1.17 (+3V3), R6.1; no longer U3.11 (FLT)
- net +5V: now also A1.2 (+5V), A1.4 (+5V), U1.2 (VCC)
- net GND: now also A1.14 (GND), A1.20 (GND), A1.25 (GND), A1.30 (GND), A1.34 (GND), A1.39 (GND), A1.6 (GND), A1.9 (GND), JP1.1 (A), U1.1 (GND)
- net I2S_CLK: now also R4.2
- net I2S_DATA: now also R5.2
- net I2S_WS: now also R1.1
- net USB_D_HOST_N: now also D2.4 (I/O2); no longer D2.3 (I/O2)
- net USB_D_HOST_P: now also D2.6 (I/O1); no longer D2.1 (I/O1)
- net USB_D_N: now also D2.3 (I/O2); no longer D2.4 (I/O2)
- net USB_D_P: now also D2.1 (I/O1); no longer D2.6 (I/O1)
- net V_USB_HOST: now also C2.1, D2.5 (VBUS), FB1.1; no longer J1.1 (VBUS)
- net DAC_LDO: now reaches C10.1, C9.1, U3.18 (LDOO)
- net I2S_DATA_SOC: now reaches R5.1
- net I2S_DATA_SOC: now also A1.40 (GP21)
- net DAC_CAPP: now reaches C8.1, U3.2 (CAPP)
- net DAC_CAPM: now reaches C8.2, U3.4 (CAPM)
- net DAC_OUTL_FILT: now reaches C12.1, J2.T, R7.2
- net DAC_OUTL: now reaches R7.1, U3.6 (OUTL)
- net USB_VBUS: now reaches D1.2 (A), USB1.11 (VBUS), USB1.2 (VBUS)
- net DAC_OUTR_FILT: now reaches C11.1, J2.R1, R8.2
- net I2S_CLK_SOC: now reaches R4.1
- net I2S_CLK_SOC: now also A1.12 (GP18)
- net DAC_VNEG: now reaches C5.1, U3.5 (VNEG)
- net DAC_OUTR: now reaches R8.1, U3.7 (OUTR)
- net OLED_SDA: now reaches A1.3 (GP2/SDA)
- net OLED_SDA: now also U1.4 (SDA)
- net I2S_WS_SOC: now reaches A1.35 (GP19)
- net I2S_WS_SOC: now also R1.2
- net OLED_SCL: now reaches A1.5 (GP3/SCL)
- net OLED_SCL: now also U1.3 (SCL)
- new net DAC_FLT: JP1.2 (B), R6.2, U3.11 (FLT)
- new net V_USB_HOST_FB: FB1.2, J1.1 (VBUS)
- no-connect marks 9 -> 32
Other:
- note removed: "Ferrite Bead?"
- note removed: "TODO jumper for latency?"
- moved on the sheet: C1, C10, C11, C12, C2, C3, C4, C5, C6, C7, C8, C9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

Commit message: Routed
Connections:
- net +3V3D: no longer A1.1 (+3V3)
- no-connect marks 32 -> 33
Changed lines of the file:
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@@
-	)
-	(junction
-		(at 50.8 110.49)
-		(diameter 0)
-		(color 0 0 0 0)
 	)
 	(junction
@@
 	)
 	(no_connect
+		(at 54.61 110.49)
+	)
+	(no_connect
 		(at 50.8 38.1)
 	)
@@
 	(wire
 		(pts
-			(xy 50.8 110.49) (xy 50.8 101.6)
+			(xy 50.8 101.6) (xy 50.8 130.81)
 		)
 		(stroke
@@
 	(wire
 		(pts
-			(xy 50.8 130.81) (xy 50.8 110.49)
-		)
-		(stroke
-			(width 0)
-			(type default)
-		)
-	)
-	(wire
-		(pts
 			(xy 38.1 118.11) (xy 41.91 118.11)
 		)
@@
 		)
 		(stroke
-			(width 0)
-			(type default)
-		)
-	)
-	(wire
-		(pts
-			(xy 54.61 110.49) (xy 50.8 110.49)
-		)
-		(stroke

Commit message: First attempt at fab files
Parts:
- A1, U1: now left out of the parts list
- C11, C12: footprint Capacitor_SMD:C_0402_1005Metric -> Capacitor_SMD:C_0805_2012Metric; LCSC Part (none) -> C28260
- J1: LCSC Part (none) -> C42474
- J2: LCSC Part (none) -> C668606
- R1, R4, R5: LCSC Part (none) -> C25092
- R7, R8: LCSC Part (none) -> C25117
- U3: LCSC Part (none) -> C107671
Other:
- note removed: "COG"
Changed lines of the file:
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@@
 	(generator_version "9.0")
 	(paper "A4")
-	(text "COG"
-		(exclude_from_sim no)
-		(at 242.57 90.17 0)
-		(effects
-			(font
-				(size 1.27 1.27)
-			)
-		)
-	)
 	(junction
 		(at 193.04 66.04)
@@
 		(unit 1)
 		(exclude_from_sim no)
-		(in_bom yes)
+		(in_bom no)
 		(on_board yes)
 		(dnp no)
@@
 			)
 		)
-		(property "LCSC Part" ""
+		(property "LCSC Part" "C25092"
 			(at 101.6 127 0)
 			(effects
@@
 			)
 		)
-		(property "Footprint" "Capacitor_SMD:C_0402_1005Metric"
+		(property "Footprint" "Capacitor_SMD:C_0805_2012Metric"
 			(at 240.9952 97.79 0)
 			(effects
@@
 			)
 		)
-		(property "LCSC Part" ""
+		(property "LCSC Part" "C28260"
 			(at 240.03 93.98 0)
 			(effects
@@
 			)
 		)
-		(property "LCSC Part" ""
+		(property "LCSC Part" "C25117"
 			(at 226.06 82.55 0)
 			(effects
@@
 			)
 		)
+		(property "LCSC Part" "C42474"
+			(at 152.4 163.83 0)
+			(effects
+				(font
+					(size 1.27 1.27)
+				)
+				(hide yes)
+			)
+		)
 		(pin "5"
 		)
@@
 			)
 		)
-		(property "Footprint" "Capacitor_SMD:C_0402_1005Metric"
+		(property "Footprint" "Capacitor_SMD:C_0805_2012Metric"
 			(at 233.9848 97.79 0)
 			(effects
@@
 			)
 		)
-		(property "LCSC Part" ""
+		(property "LCSC Part" "C28260"
 			(at 234.95 93.98 0)
 			(effects
@@
 			)
 		)
+		(property "LCSC Part" "C668606"
+			(at 259.08 87.63 0)
+			(effects
+				(font
+					(size 1.27 1.27)
+				)
+				(hide yes)
+			)
+		)
 		(pin "R1"
 		)
@@
 			)
 		)
-		(property "LCSC Part" ""
+		(property "LCSC Part" "C25092"
 			(at 101.6 123.19 0)
 			(effects
@@
 			)
 		)
-		(property "LCSC Part" ""
+		(property "LCSC Part" "C25117"
 			(at 226.06 85.09 0)
 			(effects
@@
 			)
 		)
+		(property "LCSC Part" "C107671"
+			(at 186.69 92.71 0)
+			(effects
+				(font
+					(size 1.27 1.27)
+				)
+				(hide yes)
+			)
+		)
 		(pin "18"
 		)
@@
 		(unit 1)
 		(exclude_from_sim no)
-		(in_bom yes)
+		(in_bom no)
 		(on_board yes)
 		(dnp no)
@@
 			)
 		)
-		(property "LCSC Part" ""
+		(property "LCSC Part" "C25092"
 			(at 38.1 153.67 0)
 			(effects
